Commit message: Added inertial properties of links with macro taken from franka_ros.

File: my_panda_description/robots/panda_arm.urdf.xacro (robot description, xacro)
@@ -8,5 +8,5 @@
   <xacro:arg name="use_sim" default="false" />
   <xacro:arg name="simulation_controllers_config_file"
-    default="$(find my_panda_controller)/config/joint_controller_manipulation.yaml" />
+    default="$(find my_panda_controller)/config/panda_ros_controllers.yaml" />
   <!-- box shaped table as base -->
   <link name="base">
@@ -28,5 +28,5 @@
   </link>
   <xacro:include filename="$(find my_panda_description)/robots/panda_arm.xacro" />
-  <xacro:panda_arm arm_id="$(arg arm_id)" connected_to="base" xyz="0 0 1" safety_distance="0.03" />
+  <xacro:panda_arm arm_id="$(arg arm_id)" use_sim="$(arg use_sim)" connected_to="base" xyz="0 0 1" safety_distance="0.03" />
   <xacro:if value="$(arg hand)">
     <xacro:include filename="$(find my_panda_description)/robots/hand.xacro" />

File: my_panda_description/robots/panda_arm.xacro (robot description, xacro)
@@ -5,6 +5,30 @@
   <!-- arm_id: Namespace of the panda arm. Serves to differentiate between arms in case of multiple
   instances. -->
+  <!-- Load inertial properties. Property is implicitly passed to macros. -->
+  <xacro:property name="inertial_config"
+    value="$(find my_panda_description)/robots/common/inertial.yaml" />
+  <xacro:property name="inertial" value="${xacro.load_yaml(inertial_config)}" />
+  <!-- ============================================================== -->
+  <!-- Macro to add an <inertial> tag based on yaml-load properties   -->
+  <!--                                                                -->
+  <!-- name:     Name of the robot link (without prefix)              -->
+  <!-- inertial: Dictionary of inertia properties (see inertial.yaml) -->
+  <!-- ============================================================== -->
+  <xacro:macro name="inertial_props" params="name inertial:=^">
+    <xacro:unless value="${name in inertial}">${xacro.warning('No inertia properties defined for: '
+      + name)}</xacro:unless>
+    <xacro:if value="${name in inertial}">
+      <!-- Access inertia properties of link 'name' -->
+      <xacro:property name="inertial" value="${inertial[name]}" lazy_eval="false" />
+      <inertial>
+        <origin rpy="${inertial.origin.rpy}" xyz="${inertial.origin.xyz}" />
+        <mass value="${inertial.mass}" />
+        <xacro:property name="I" value="${inertial.inertia}" />
+        <inertia ixx="${I.xx}" ixy="${I.xy}" ixz="${I.xz}" iyy="${I.yy}" iyz="${I.yz}" izz="${I.zz}" />
+      </inertial>
+    </xacro:if>
+  </xacro:macro>
   <xacro:macro name="panda_arm"
-    params="arm_id:='panda' description_pkg:='franka_description' connected_to:='' xyz:='0 0 0' rpy:='0 0 0' safety_distance:=0">
+    params="arm_id:='panda' use_sim:='false' description_pkg:='franka_description' connected_to:='' xyz:='0 0 0' rpy:='0 0 0' safety_distance:=0">
     <xacro:unless value="${not connected_to}">
       <joint name="${arm_id}_joint_${connected_to}" type="fixed">
@@ -63,4 +87,7 @@
         </geometry>
       </collision>
+      <xacro:if value="${use_sim}">
+        <xacro:inertial_props name="link1" />
+      </xacro:if>
     </link>
     <joint name="${arm_id}_joint1" type="revolute">
@@ -97,4 +124,7 @@
         </geometry>
       </collision>
+      <xacro:if value="${use_sim}">
+        <xacro:inertial_props name="link2" />
+      </xacro:if>
     </link>
     <joint name="${arm_id}_joint2" type="revolute">
@@ -131,4 +161,7 @@
         </geometry>
       </collision>
+      <xacro:if value="${use_sim}">
+        <xacro:inertial_props name="link3" />
+      </xacro:if>
     </link>
     <joint name="${arm_id}_joint3" type="revolute">
@@ -165,4 +198,7 @@
         </geometry>
       </collision>
+      <xacro:if value="${use_sim}">
+        <xacro:inertial_props name="link4" />
+      </xacro:if>
     </link>
     <joint name="${arm_id}_joint4" type="revolute">
@@ -217,4 +253,7 @@
         </geometry>
       </collision>
+      <xacro:if value="${use_sim}">
+        <xacro:inertial_props name="link5" />
+      </xacro:if>
     </link>
     <joint name="${arm_id}_joint5" type="revolute">
@@ -251,4 +290,7 @@
         </geometry>
       </collision>
+      <xacro:if value="${use_sim}">
+        <xacro:inertial_props name="link6" />
+      </xacro:if>
     </link>
     <joint name="${arm_id}_joint6" type="revolute">
@@ -285,4 +327,7 @@
         </geometry>
       </collision>
+      <xacro:if value="${use_sim}">
+        <xacro:inertial_props name="link7" />
+      </xacro:if>
     </link>
     <joint name="${arm_id}_joint7" type="revolute">

File: my_panda_description/robots/ros2_control/panda_arm.ros2_control.xacro (robot description, xacro)
@@ -1,47 +1,63 @@
 <?xml version="1.0"?>
 <robot xmlns:xacro="http://www.ros.org/wiki/xacro">
+  <!-- Include Utils xacro -->
+  <xacro:include filename="$(find my_panda_description)/robots/ros2_control/utils.xacro" />
   <xacro:macro name="panda_arm_ros2_control"
     params="ns use_sim simulation_controllers_config_file robot_ip use_fake_hardware:=^|false fake_sensor_commands:=^|false">
-    <ros2_control name="FrankaHardwareInterface" type="system">
-      <hardware>
-        <xacro:if value="${use_fake_hardware}">
-          <plugin>fake_components/GenericSystem</plugin>
-          <param name="fake_sensor_commands">${fake_sensor_commands}</param>
-          <param name="state_following_offset">0.0</param>
-        </xacro:if>
-        <xacro:unless value="${use_fake_hardware}">
-          <plugin>franka_hardware/FrankaHardwareInterface</plugin>
-          <param name="robot_ip">${robot_ip}</param>
-        </xacro:unless>
-      </hardware>
-      <xacro:macro name="configure_joint" params="joint_name initial_position">
-        <joint name="${joint_name}">
-          <param name="initial_position">${initial_position}</param>
-          <command_interface name="effort" />
-          <command_interface name="velocity" />
-          <command_interface name="position" />
-          <state_interface name="position" />
-          <state_interface name="velocity" />
-          <state_interface name="effort" />
-        </joint>
-      </xacro:macro>
-      <xacro:configure_joint joint_name="${ns}_joint1" initial_position="0.0" />
-      <xacro:configure_joint joint_name="${ns}_joint2" initial_position="${-pi/4}" />
-      <xacro:configure_joint joint_name="${ns}_joint3" initial_position="0.0" />
-      <xacro:configure_joint joint_name="${ns}_joint4" initial_position="${-3*pi/4}" />
-      <xacro:configure_joint joint_name="${ns}_joint5" initial_position="0.0" />
-      <xacro:configure_joint joint_name="${ns}_joint6" initial_position="${pi/2}" />
-      <xacro:configure_joint joint_name="${ns}_joint7" initial_position="${pi/4}" />
-      <xacro:if value="$(arg use_sim)">
+    <xacro:unless value="$(arg use_sim)">
+      <ros2_control name="FrankaHardwareInterface" type="system">
+        <hardware>
+          <xacro:if value="${use_fake_hardware}">
+            <plugin>fake_components/GenericSystem</plugin>
+            <param name="fake_sensor_commands">${fake_sensor_commands}</param>
+            <param name="state_following_offset">0.0</param>
+          </xacro:if>
+          <xacro:unless value="${use_fake_hardware}">
+            <plugin>franka_hardware/FrankaHardwareInterface</plugin>
+            <param name="robot_ip">${robot_ip}</param>
+          </xacro:unless>
+        </hardware>
+        <xacro:configure_joint joint_name="${ns}_joint1" initial_position="0.0" />
+        <xacro:configure_joint joint_name="${ns}_joint2" initial_position="${-pi/4}" />
+        <xacro:configure_joint joint_name="${ns}_joint3" initial_position="0.0" />
+        <xacro:configure_joint joint_name="${ns}_joint4" initial_position="${-3*pi/4}" />
+        <xacro:configure_joint joint_name="${ns}_joint5" initial_position="0.0" />
+        <xacro:configure_joint joint_name="${ns}_joint6" initial_position="${pi/2}" />
+        <xacro:configure_joint joint_name="${ns}_joint7" initial_position="${pi/4}" />
+      </ros2_control>
+    </xacro:unless>
+    <xacro:if value="$(arg use_sim)">
+      <ros2_control name="FrankaHardwareInterface" type="system">
+        <hardware>
+          <xacro:if value="${use_fake_hardware}">
+            <plugin>fake_components/GenericSystem</plugin>
+            <param name="fake_sensor_commands">${fake_sensor_commands}</param>
+            <param name="state_following_offset">0.0</param>
+          </xacro:if>
+          <xacro:unless value="${use_fake_hardware}">
+            <plugin>franka_hardware/FrankaHardwareInterface</plugin>
+            <param name="robot_ip">${robot_ip}</param>
+          </xacro:unless>
+        </hardware>
+        <xacro:configure_joint joint_name="${ns}_joint1" initial_position="0.0" />
+        <xacro:configure_joint joint_name="${ns}_joint2" initial_position="${-pi/4}" />
+        <xacro:configure_joint joint_name="${ns}_joint3" initial_position="0.0" />
+        <xacro:configure_joint joint_name="${ns}_joint4" initial_position="${-3*pi/4}" />
+        <xacro:configure_joint joint_name="${ns}_joint5" initial_position="0.0" />
+        <xacro:configure_joint joint_name="${ns}_joint6" initial_position="${pi/2}" />
+        <xacro:configure_joint joint_name="${ns}_joint7" initial_position="${pi/4}" />
         <hardware>
           <plugin>ign_ros2_control/IgnitionSystem</plugin>
         </hardware>
-      </xacro:if>
-    </ros2_control>
+      </ros2_control>
+    </xacro:if>
     <!-- Joint state publisher -->
     <xacro:if value="$(arg use_sim)">
-      <plugin filename="ign_ros2_control-system" name="ign_ros2_control::IgnitionROS2ControlPlugin">
-        <parameters>${simulation_controllers_config_file}</parameters>
-      </plugin>
+      <gazebo>
+        <plugin filename="ign_ros2_control-system"
+          name="ign_ros2_control::IgnitionROS2ControlPlugin">
+          <parameters>${simulation_controllers_config_file}</parameters>
+        </plugin>
+      </gazebo>
     </xacro:if>
   </xacro:macro>
